Commit message: fixed camera transformations

File: ROS_ws/src/custom_slam/urdf/realsense.xacro (robot description, xacro)
@@ -11,53 +11,53 @@
   <link name="camera_right_ir_frame"></link>
   <link name="camera_right_ir_optical_frame"></link>
-   <joint name="camera_joint" type="fixed">
+  <joint name="camera_joint" type="fixed">
     <parent link="base_link" />
     <child link="camera_bottom_screw_frame" />
-    <pose xyz="0.4 0 0.05" rpy="0 0 0" />
+    <origin xyz="0.4 0 0.05" rpy="0 0 0" />
   </joint>
   <joint name="camera_link_joint" type="fixed">
     <parent link="camera_bottom_screw_frame" />
     <child link="camera_link" />
-    <pose xyz="0.3 0 0" rpy="0 0 0" />
+    <origin xyz="0.3 0 0" rpy="0 0 0" />
   </joint>
   <joint name="camera_depth_joint" type="fixed">
     <parent link="camera_link" />
     <child link="camera_depth_frame" />
-    <pose xyz="0 0 0" rpy="0 0 0" />
+    <origin xyz="0 0 0" rpy="0 0 0" />
   </joint>
   <joint name="camera_depth_optical_joint" type="fixed">
     <parent link="camera_depth_frame" />
     <child link="camera_depth_optical_frame" />
-    <pose xyz="0 0 0 " rpy="-1.57 0 -1.57" />
+    <origin xyz="0 0 0 " rpy="-1.57 0 -1.57" />
   </joint>
   <joint name="camera_color_joint" type="fixed">
     <parent link="camera_depth_frame" />
     <child link="camera_color_frame" />
-    <pose xyz="0 0 0" rpy="0 0 0" />
+    <origin xyz="0 0 0" rpy="0 0 0" />
   </joint>
   <joint name="camera_color_optical_joint" type="fixed">
     <parent link="camera_color_frame" />
     <child link="camera_color_optical_frame" />
-    <pose xyz="0 0 0 " rpy="-1.57 0 -1.57" />
+    <origin xyz="0 0 0 " rpy="-1.57 0 -1.57" />
   </joint>
   <joint name="camera_left_ir_joint" type="fixed">
     <parent link="camera_depth_frame" />
     <child link="camera_left_ir_frame" />
-    <pose xyz="0 0 0 " rpy="0 0 0 " />
+    <origin xyz="0 0 0 " rpy="0 0 0 " />
   </joint>
   <joint name="camera_left_ir_optical_joint" type="fixed">
     <parent link="camera_left_ir_frame" />
     <child link="camera_left_ir_optical_frame" />
-    <pose xyz="0 0 0 " rpy="-1.57 0 -1.57" />
+    <origin xyz="0 0 0 " rpy="-1.57 0 -1.57" />
   </joint>
   <joint name="camera_right_ir_joint" type="fixed">
     <parent link="camera_depth_frame" />
     <child link="camera_right_ir_frame" />
-    <pose xyz="0 -0.050 0 " rpy="0 0 0" />
+    <origin xyz="0 -0.050 0 " rpy="0 0 0" />
   </joint>
   <joint name="camera_right_ir_optical_joint" type="fixed">
     <parent link="camera_right_ir_frame" />
     <child link="camera_right_ir_optical_frame" />
-    <pose xyz="0 0 0 " rpy="-1.57 0 -1.57" />
+    <origin xyz="0 0 0 " rpy="-1.57 0 -1.57" />
   </joint>
   <!-- Realsense link -->
@@ -110,5 +110,5 @@
       </camera>
       <always_on>1</always_on>
-      <update_rate>30</update_rate>
+      <update_rate>60</update_rate>
       <visualize>0</visualize>
     </sensor>
@@ -134,5 +134,5 @@
       </camera>
       <always_on>1</always_on>
-      <update_rate>30</update_rate>
+      <update_rate>60</update_rate>
       <visualize>1</visualize>
     </sensor>
@@ -190,6 +190,6 @@
     <plugin name="camera" filename="librealsense_gazebo_plugin.so">
       <prefix>camera</prefix>
-      <depthUpdateRate>30.0</depthUpdateRate>
-      <colorUpdateRate>30.0</colorUpdateRate>
+      <depthUpdateRate>60.0</depthUpdateRate>
+      <colorUpdateRate>60.0</colorUpdateRate>
       <infraredUpdateRate>1.0</infraredUpdateRate>
       <depthTopicName>aligned_depth_to_color/image_raw</depthTopicName>
