Commit message: fixed odometry

File: ROS_ws/src/custom_slam/urdf/osr_full.urdf.xacro (robot description, xacro)
@@ -50,5 +50,5 @@
             <origin rpy="0 0 -3.14" xyz="0 0 0.0"/>
             <geometry>
-                    <box size="0.2 0.1 0.05"/>
+                <box size="0.2 0.1 0.05"/>
             </geometry>
         </collision>
@@ -225,5 +225,5 @@
                 <origin rpy="0 0 ${dir*-1.57}" xyz="0 0 0.0"/>
                 <geometry>
-                    <mesh filename="file://$(find custom_slam)/meshes/wheel_link_left_2.stl"/>
+                    <box size="0.2 0.1 0.05"/>
                 </geometry>
             </collision>
@@ -253,5 +253,5 @@
                 <origin rpy="${origin} 0 ${-dir*1.57}" xyz="0 0 0.0"/>
                 <geometry>
-                    <mesh filename="file://$(find custom_slam)/meshes/wheel_middle_left.stl"/>
+                    <box size="0.2 0.1 0.05"/>
                 </geometry>
             </collision>
@@ -279,5 +279,5 @@
                 <origin rpy="0 0 ${-dir*1.57}" xyz="0 0 0.0"/>
                 <geometry>
-                    <mesh filename="file://$(find custom_slam)/meshes/wheel_link_left_2.stl"/>
+                    <box size="0.2 0.1 0.05"/>
                 </geometry>
             </collision>
@@ -311,5 +311,5 @@
                 <origin rpy="-1.57 0 ${origin}" xyz="0 0 0.0"/>
                 <geometry>
-                    <mesh filename="file://$(find custom_slam)/meshes/wheel.stl"/>
+                    <cylinder radius="0.0675" length="0.052"/>
                 </geometry>
                 <surface>
@@ -346,5 +346,5 @@
                 <origin rpy="-1.57 0 ${origin}" xyz="0 0 0.0"/>
                 <geometry>
-                    <mesh filename="file://$(find custom_slam)/meshes/wheel.stl"/>
+                    <cylinder radius="0.0675" length="0.052"/>
                 </geometry>
                 <surface>
@@ -381,5 +381,5 @@
                 <origin rpy="-1.57 0 ${origin}" xyz="0 0 0.0"/>
                 <geometry>
-                    <mesh filename="file://$(find custom_slam)/meshes/wheel.stl"/>
+                    <cylinder radius="0.0675" length="0.052"/>
                 </geometry>
                 <surface>

Commit message: BEV Builder and Matcher work

File: ROS_ws/src/custom_slam/urdf/osr_full.urdf.xacro (robot description, xacro)
@@ -311,11 +311,11 @@
                 <origin rpy="-1.57 0 ${origin}" xyz="0 0 0.0"/>
                 <geometry>
-                    <cylinder radius="0.0675" length="0.052"/>
+                    <cylinder radius="0.075" length="0.052"/>
                 </geometry>
                 <surface>
                     <friction>
                         <ode>
-                            <mu>0.7</mu>
-                            <mu2>0.3</mu2>
+                            <mu>3.7</mu>
+                            <mu2>3.3</mu2>
                         </ode>
                     </friction>
@@ -346,11 +346,11 @@
                 <origin rpy="-1.57 0 ${origin}" xyz="0 0 0.0"/>
                 <geometry>
-                    <cylinder radius="0.0675" length="0.052"/>
+                    <cylinder radius="0.075" length="0.052"/>
                 </geometry>
                 <surface>
                     <friction>
                         <ode>
-                            <mu>0.7</mu>
-                            <mu2>0.3</mu2>
+                            <mu>3.7</mu>
+                            <mu2>3.3</mu2>
                         </ode>
                     </friction>
@@ -381,11 +381,11 @@
                 <origin rpy="-1.57 0 ${origin}" xyz="0 0 0.0"/>
                 <geometry>
-                    <cylinder radius="0.0675" length="0.052"/>
+                    <cylinder radius="0.075" length="0.052"/>
                 </geometry>
                 <surface>
                     <friction>
                         <ode>
-                            <mu>0.7</mu>
-                            <mu2>0.3</mu2>
+                            <mu>3.7</mu>
+                            <mu2>3.3</mu2>
                         </ode>
                     </friction>

Commit message: Mapper has errors in rock duplication

File: ROS_ws/src/custom_slam/urdf/osr_full.urdf.xacro (robot description, xacro)
@@ -437,5 +437,5 @@
         <parent link="camera_link"/>
         <child link="left_camera_frame"/>
-        <origin xyz="0 0.035 0" rpy="0 0 0"/>  <!-- +35mm left -->
+        <origin xyz="0 0.05 0" rpy="0 0 0"/>  <!-- +35mm left -->
     </joint>
     <link name="left_camera_frame"/>
@@ -450,5 +450,5 @@
         <parent link="camera_link"/>
         <child link="right_camera_frame"/>
-        <origin xyz="0 -0.035 0" rpy="0 0 0"/>  <!-- -35mm right -->
+        <origin xyz="0 -0.05 0" rpy="0 0 0"/>  <!-- -35mm right -->
     </joint>
     <link name="right_camera_frame"/>

Commit message: full pipeline works

File: ROS_ws/src/custom_slam/urdf/osr_full.urdf.xacro (robot description, xacro)
@@ -437,5 +437,5 @@
         <parent link="camera_link"/>
         <child link="left_camera_frame"/>
-        <origin xyz="0 0.05 0" rpy="0 0 0"/>  <!-- +35mm left -->
+        <origin xyz="0 0.05 0" rpy="0 0.261799 0"/> <!-- +35mm left -->
     </joint>
     <link name="left_camera_frame"/>
@@ -450,5 +450,5 @@
         <parent link="camera_link"/>
         <child link="right_camera_frame"/>
-        <origin xyz="0 -0.05 0" rpy="0 0 0"/>  <!-- -35mm right -->
+        <origin xyz="0 -0.05 0" rpy="0 0.261799 0"/>  <!-- -35mm right -->
     </joint>
     <link name="right_camera_frame"/>

Commit message: timing problems sorta fixed

File: ROS_ws/src/custom_slam/urdf/osr_full.urdf.xacro (robot description, xacro)
@@ -467,5 +467,5 @@
         <parent link="camera_link"/>
         <child link="left_camera_frame"/>
-        <origin xyz="0 0.05 0" rpy="0 0.261799 0"/> <!-- +35mm left -->
+        <origin xyz="0 0.05 0" rpy="0 0.261799 0"/>
     </joint>
     <link name="left_camera_frame"/>
@@ -480,5 +480,5 @@
         <parent link="camera_link"/>
         <child link="right_camera_frame"/>
-        <origin xyz="0 -0.05 0" rpy="0 0.261799 0"/>  <!-- -35mm right -->
+        <origin xyz="0 -0.05 0" rpy="0 0.261799 0"/>
     </joint>
     <link name="right_camera_frame"/>
