Commit message: realsense camera integration to gazebo sim

File: ROS_ws/src/custom_slam/urdf/gazebo.urdf.xacro (robot description, xacro)
@@ -120,5 +120,5 @@
     </plugin>
   </gazebo>
-  <!-- IMU Sensor
+  <!-- IMU Sensor -->
   <gazebo reference="imu_link">
     <gravity>true</gravity>
@@ -138,5 +138,5 @@
       </plugin>
     </sensor>
-  </gazebo> -->
+  </gazebo>
   <!-- LiDAR Sensor
   <gazebo reference="lidar_link">
@@ -169,40 +169,3 @@
   </gazebo> -->
   <!-- Camera Sensor -->
-  <gazebo reference="zed_camera_link">
-    <sensor name="zed_camera" type="camera">
-      <visualize>true</visualize>
-      <pose>0.2 0.0 0 0 0 0</pose>  <!-- Position the camera (adjust if needed) -->
-      <camera name="camera">
-        <horizontal_fov>2.09</horizontal_fov>  <!-- Field of view of ZED 2i -->
-        <image>
-          <width>2688</width>  <!-- Camera resolution (set to ZED 2i default) -->
-          <height>1520</height>
-          <format>R8G8B8</format>
-        </image>
-        <depth>
-          <width>1280</width>
-          <height>720</height>
-        </depth>
-        <clip>
-          <near>0.1</near>  <!-- Near clipping distance -->
-          <far>3</far>     <!-- Far clipping distance -->
-        </clip>
-        <update_rate>30.0</update_rate>  <!-- Frame rate of the camera -->
-      </camera>
-      <plugin name="gazebo_ros_camera" filename="libgazebo_ros_camera.so">
-        <frame_name>zed_camera_link</frame_name>  <!-- Link to which the camera is attached -->
-        <alwaysOn>true</alwaysOn>
-        <ros>
-          <remapping>/camera/image_raw:=/zed_camera/image_raw</remapping>  <!-- Remap topics if needed -->
-        </ros>
-        <camera_name>zed_camera</camera_name>
-        <image_topic>/camera/image_raw</image_topic>
-        <depth_topic>/camera/depth_raw</depth_topic>
-        <point_cloud_topic>/camera/point_cloud</point_cloud_topic>  <!-- Optional for depth camera -->
-        <frame_name>zed_camera_link</frame_name>
-        <always_on>true</always_on>
-        <update_rate>30.0</update_rate>  <!-- Camera update rate -->
-      </plugin>
-    </sensor>
-  </gazebo>
 </robot>

File: ROS_ws/src/custom_slam/urdf/osr.urdf.xacro (robot description, xacro)
@@ -18,4 +18,5 @@
     <xacro:include filename="$(find custom_slam)/urdf/gazebo.urdf.xacro"/>
     <xacro:include filename="$(find custom_slam)/urdf/insert_transmission.urdf.xacro"/>
+    <xacro:include filename="$(find custom_slam)/urdf/realsense.xacro"/>
     <link name="base_footprint"/>
     <link name="base_link">
@@ -430,27 +431,3 @@
     <xacro:insert_position_transmission name="rear_wheel_joint_R"/>
     <xacro:insert_position_transmission name="rear_wheel_joint_L"/>
-  <!-- Camera Link -->
-  <link name="zed_camera_link">
-    <visual>
-      <geometry>
-        <box size="0.1 0.1 0.1"/>  <!-- Adjust the size based on your model -->
-      </geometry>
-      <material name="blue"/>
-    </visual>
-    <collision>
-      <geometry>
-        <box size="0.1 0.1 0.1"/>
-      </geometry>
-    </collision>
-    <inertial>
-      <mass value="0.1"/>
-      <inertia ixx="0.001" ixy="0.0" ixz="0.0" iyy="0.001" iyz="0.0" izz="0.001"/>
-    </inertial>
-  </link>
-  <!-- Camera Joint (if you need it to be movable, like on a pan/tilt setup) -->
-  <joint name="zed_camera_joint" type="fixed">
-    <parent link="base_link"/>
-    <child link="zed_camera_link"/>
-    <origin xyz="0.2 0.0 0.0" rpy="0 0 0"/>
-  </joint>
 </robot>

Commit message: Working rock identifier

File: ROS_ws/src/custom_slam/urdf/gazebo.urdf.xacro (robot description, xacro)
@@ -1,10 +1,11 @@
 <?xml version="1.0"?>
-<robot xmlns:xacro="http://wiki.ros.org/xacro">
-  <!-- ROS 2 Control Configuration -->
+<robot name="my_robot" xmlns:xacro="http://wiki.ros.org/xacro">
+  <!-- ros2_control configuration -->
   <ros2_control name="GazeboSystem" type="system">
     <hardware>
-      <plugin>gazebo_ros2_control/GazeboSystem</plugin>
+      <!-- Gazebo Harmonic ros2_control hardware plugin -->
+      <plugin>gz_ros2_control/GazeboSimSystem</plugin>
     </hardware>
-    <!-- Joints -->
+    <!-- Wheel joints (unchanged) -->
     <joint name="middle_wheel_joint_left">
       <command_interface name="velocity">
@@ -60,5 +61,5 @@
       <state_interface name="effort"/>
     </joint>
-    <!-- Front and Rear Rotating Joints -->
+    <!-- Steering/rotating joints (unchanged) -->
     <joint name="front_wheel_joint_R">
       <command_interface name="position">
@@ -113,38 +114,64 @@
       <state_interface name="effort"/>
     </joint>
+    <!-- Rocker-bogie joints -->
+    <joint name="rocker_bogie_joint_L_2">
+        <command_interface name="effort"/>
+        <state_interface name="position"/>
+        <state_interface name="velocity"/>
+        <state_interface name="effort"/>
+    </joint>
+    <joint name="rocker_bogie_joint_R_2">
+        <command_interface name="effort"/>
+        <state_interface name="position"/>
+        <state_interface name="velocity"/>
+        <state_interface name="effort"/>
+    </joint>
   </ros2_control>
-  <!-- Gazebo Plugin -->
-  <gazebo>
-    <plugin filename="libgazebo_ros2_control.so" name="gazebo_ros2_control">
-      <parameters>$(find custom_slam)/config/controller_velocity.yaml</parameters>
-    </plugin>
+  <!-- Gazebo Harmonic ros2_control system plugin -->
+<gazebo>
+  <plugin filename="libgz_ros2_control-system.so" name="gz_ros2_control::GazeboSimROS2ControlPlugin">
+    <parameters>$(find custom_slam)/config/controller_velocity.yaml</parameters>
+  </plugin>
+</gazebo>
+<gazebo>
+  <plugin filename="gz-sim-odometry-publisher-system"
+          name="gz::sim::systems::OdometryPublisher">
+    <!-- Frame IDs -->
+    <odom_frame>odom</odom_frame>
+    <robot_base_frame>base_footprint</robot_base_frame>
+    <!-- Publishing settings -->
+    <odom_publish_frequency>50</odom_publish_frequency>
+    <odom_topic>/ground_truth/odom</odom_topic>
+    <!-- Ground truth mode - no noise or drift -->
+    <xyz_offset>0 0 0</xyz_offset>
+    <rpy_offset>0 0 0</rpy_offset>
+    <!-- Gaussian noise (set to 0 for perfect ground truth) -->
+    <gaussian_noise>0.0</gaussian_noise>
+  </plugin>
+</gazebo>
+  <!-- Sensors (URDF -> SDF extension through <gazebo reference="...">) -->
+  <!-- IMU on imu_link -->
+  <gazebo reference="imu_link">
+    <sensor name="tb3_imu" type="imu">
+      <always_on>true</always_on>
+      <update_rate>200</update_rate>
+      <topic>imu</topic>
+      <gz_frame_id>imu_link</gz_frame_id>
+      <frame_id>imu_link</frame_id>
+      <!-- Optional: orientation reference / noise can be added here -->
+    </sensor>
   </gazebo>
-  <!-- IMU Sensor -->
-  <gazebo reference="imu_link">
-    <gravity>true</gravity>
-    <sensor name="imu_sensor" type="imu">
+  <!-- GPU LiDAR on lidar_link -->
+  <!-- <gazebo reference="base_scan">
+    <sensor type="gpu_lidar" name="lidar_sensor">
       <always_on>true</always_on>
-      <update_rate>100</update_rate>
       <visualize>true</visualize>
-      <plugin filename="libgazebo_ros_imu_sensor.so" name="imu_plugin">
-        <topicName>imu</topicName>
-        <bodyName>imu_link</bodyName>
-        <updateRateHZ>100.0</updateRateHZ>
-        <gaussianNoise>0.0</gaussianNoise>
-        <xyzOffset>0 0 0</xyzOffset>
-        <rpyOffset>0 0 0</rpyOffset>
-        <frameName>imu_link</frameName>
-        <initialOrientationAsReference>false</initialOrientationAsReference>
-      </plugin>
-    </sensor>
-  </gazebo>
-  <!-- LiDAR Sensor
-  <gazebo reference="lidar_link">
-    <sensor type="ray" name="lidar_sensor">
-      <always_on>true</always_on>
-      <pose>0 0 0 0 0 0</pose>
-      <update_rate>20.0</update_rate>
-      <visualize>true</visualize>
-      <ray>
+      <pose>-0.064 0 0.121 0 0 0</pose>
+      <update_rate>20</update_rate>
+      <topic>scan</topic>
+      <!- Header frame id used in gz msgs; bridge to ROS if needed ->
+      <frame_id>base_scan</frame_id>
+      <gz_frame_id>base_scan</gz_frame_id>
+      <lidar>
         <scan>
           <horizontal>
@@ -157,15 +184,55 @@
         <range>
           <min>0.2</min>
-          <max>30.0</max>
-          <resolution>0.01</resolution>
+          <max>10.0</max>
+          <resolution>1</resolution>
         </range>
-      </ray>
-    <plugin name="scan" filename="libgazebo_ros_laser.so">
-      <bodyName>scan</bodyName>
-      <topicName>scan</topicName> Topic for publishing scan data
-      <frameName>lidar_link</frameName> Reference frame
-    </plugin>
+      </lidar>
+      <ros>
+        <frame_name>base_scan</frame_name>
+      </ros>
     </sensor>
   </gazebo> -->
-  <!-- Camera Sensor -->
+<gazebo reference="left_camera_frame">
+    <sensor name="left_camera" type="camera">
+        <always_on>true</always_on>
+        <update_rate>30</update_rate>
+        <topic>left_camera/image_raw</topic>
+        <gz_frame_id>left_camera_optical_frame</gz_frame_id>
+        <frame_id>left_camera_optical_frame</frame_id>
+        <camera>
+            <horizontal_fov>1.0472</horizontal_fov>
+            <image>
+                <width>2304</width>
+                <height>1296</height>
+                <format>R8G8B8</format>
+            </image>
+            <clip>
+                <near>0.01</near>
+                <far>100</far>
+            </clip>
+        </camera>
+    </sensor>
+</gazebo>
+<gazebo reference="right_camera_frame">
+    <sensor name="right_camera" type="camera">
+        <always_on>true</always_on>
+        <update_rate>30</update_rate>
+        <topic>right_camera/image_raw</topic>
+        <gz_frame_id>right_camera_optical_frame</gz_frame_id>
+        <frame_id>right_camera_optical_frame</frame_id>
+        <camera>
+            <horizontal_fov>1.0472</horizontal_fov>
+            <anti_aliasing>0</anti_aliasing>
+            <image>
+                <width>2304</width>
+                <height>1296</height>
+                <format>R8G8B8</format>
+            </image>
+            <clip>
+                <near>0.01</near>
+                <far>100</far>
+            </clip>
+        </camera>
+    </sensor>
+</gazebo>
 </robot>

File: ROS_ws/src/custom_slam/urdf/osr_full.urdf.xacro (robot description, xacro)
@@ -18,5 +18,5 @@
     <xacro:include filename="$(find custom_slam)/urdf/gazebo.urdf.xacro"/>
     <xacro:include filename="$(find custom_slam)/urdf/insert_transmission.urdf.xacro"/>
-    <xacro:include filename="$(find custom_slam)/urdf/realsense.xacro"/>
+    <!-- <xacro:include filename="$(find custom_slam)/urdf/realsense.xacro"/> -->
     <link name="base_footprint"/>
     <link name="base_link">
@@ -421,13 +421,108 @@
         </joint>
     <link name="imu_link"></link>
-    <xacro:insert_velocity_transmission name="rear_wheel_joint_right"/>
-    <xacro:insert_velocity_transmission name="rear_wheel_joint_left"/>
-    <xacro:insert_velocity_transmission name="middle_wheel_joint_right"/>
-    <xacro:insert_velocity_transmission name="middle_wheel_joint_left"/>
-    <xacro:insert_velocity_transmission name="front_wheel_joint_right"/>
-    <xacro:insert_velocity_transmission name="front_wheel_joint_left"/>
-    <xacro:insert_position_transmission name="front_wheel_joint_R"/>
-    <xacro:insert_position_transmission name="front_wheel_joint_L"/>
-    <xacro:insert_position_transmission name="rear_wheel_joint_R"/>
-    <xacro:insert_position_transmission name="rear_wheel_joint_L"/>
+    <!-- <joint name="lidar_joint" type="fixed">
+        <parent link="base_link"/>
+        <child link="base_scan"/>
+        <origin xyz="0 0 0" rpy="0 0 0"/>
+    </joint> -->
+    <!-- <link name="base_scan"></link> -->
+    <joint name="camera_joint" type="fixed">
+        <parent link="base_link"/>
+        <child link="camera_link"/>
+        <origin xyz="0 0 0.5" rpy="0 0 0"/>
+    </joint>
+    <link name="camera_link"/>
+    <!-- LEFT CAMERA -->
+    <joint name="left_camera_joint" type="fixed">
+        <parent link="camera_link"/>
+        <child link="left_camera_frame"/>
+        <origin xyz="0 0.035 0" rpy="0 0 0"/>  <!-- +35mm left -->
+    </joint>
+    <link name="left_camera_frame"/>
+    <joint name="left_camera_optical_joint" type="fixed">
+        <parent link="left_camera_frame"/>
+        <child link="left_camera_optical_frame"/>
+        <origin xyz="0 0 0" rpy="-1.570796 0 -1.570796"/>
+    </joint>
+    <link name="left_camera_optical_frame"/>
+    <!-- RIGHT CAMERA -->
+    <joint name="right_camera_joint" type="fixed">
+        <parent link="camera_link"/>
+        <child link="right_camera_frame"/>
+        <origin xyz="0 -0.035 0" rpy="0 0 0"/>  <!-- -35mm right -->
+    </joint>
+    <link name="right_camera_frame"/>
+    <joint name="right_camera_optical_joint" type="fixed">
+        <parent link="right_camera_frame"/>
+        <child link="right_camera_optical_frame"/>
+        <origin xyz="0 0 0" rpy="-1.570796 0 -1.570796"/>
+    </joint>
+    <link name="right_camera_optical_frame"/>
+    <!-- <ros2_control name="RobotSystem" type="system">
+        <hardware>
+            <plugin>gz_ros2_control/GazeboSimSystem</plugin>
+        </hardware>
+        <joint name="rear_wheel_joint_right">
+            <command_interface name="velocity"/>
+            <state_interface name="position"/>
+            <state_interface name="velocity"/>
+        </joint>
+        <joint name="rear_wheel_joint_left">
+            <command_interface name="velocity"/>
+            <state_interface name="position"/>
+            <state_interface name="velocity"/>
+        </joint>
+        <joint name="middle_wheel_joint_right">
+            <command_interface name="velocity"/>
+            <state_interface name="position"/>
+            <state_interface name="velocity"/>
+        </joint>
+        <joint name="middle_wheel_joint_left">
+            <command_interface name="velocity"/>
+            <state_interface name="position"/>
+            <state_interface name="velocity"/>
+        </joint>
+        <joint name="front_wheel_joint_right">
+            <command_interface name="velocity"/>
+            <state_interface name="position"/>
+            <state_interface name="velocity"/>
+        </joint>
+        <joint name="front_wheel_joint_left">
+            <command_interface name="velocity"/>
+            <state_interface name="position"/>
+            <state_interface name="velocity"/>
+        </joint>
+        <joint name="front_wheel_joint_R">
+            <command_interface name="position"/>
+            <state_interface name="position"/>
+            <state_interface name="velocity"/>
+        </joint>
+        <joint name="front_wheel_joint_L">
+            <command_interface name="position"/>
+            <state_interface name="position"/>
+            <state_interface name="velocity"/>
+        </joint>
+        <joint name="rear_wheel_joint_R">
+            <command_interface name="position"/>
+            <state_interface name="position"/>
+            <state_interface name="velocity"/>
+        </joint>
+        <joint name="rear_wheel_joint_L">
+            <command_interface name="position"/>
+            <state_interface name="position"/>
+            <state_interface name="velocity"/>
+        </joint>
+        <joint name="rocker_bogie_joint_L_2">
+            <command_interface name="effort"/>
+            <state_interface name="position"/>
+            <state_interface name="velocity"/>
+            <state_interface name="effort"/>
+        </joint>
+        <joint name="rocker_bogie_joint_R_2">
+            <command_interface name="effort"/>
+            <state_interface name="position"/>
+            <state_interface name="velocity"/>
+            <state_interface name="effort"/>
+        </joint>
+    </ros2_control> -->
 </robot>

Commit message: overhead mapping works from seg model

File: ROS_ws/src/custom_slam/urdf/gazebo.urdf.xacro (robot description, xacro)
@@ -137,14 +137,11 @@
   <plugin filename="gz-sim-odometry-publisher-system"
           name="gz::sim::systems::OdometryPublisher">
-    <!-- Frame IDs -->
     <odom_frame>odom</odom_frame>
     <robot_base_frame>base_footprint</robot_base_frame>
-    <!-- Publishing settings -->
     <odom_publish_frequency>50</odom_publish_frequency>
     <odom_topic>/ground_truth/odom</odom_topic>
-    <!-- Ground truth mode - no noise or drift -->
+    <tf_topic>/tf</tf_topic>
     <xyz_offset>0 0 0</xyz_offset>
     <rpy_offset>0 0 0</rpy_offset>
-    <!-- Gaussian noise (set to 0 for perfect ground truth) -->
     <gaussian_noise>0.0</gaussian_noise>
   </plugin>
@@ -163,5 +160,5 @@
   </gazebo>
   <!-- GPU LiDAR on lidar_link -->
-  <!-- <gazebo reference="base_scan">
+  <gazebo reference="base_scan">
     <sensor type="gpu_lidar" name="lidar_sensor">
       <always_on>true</always_on>
@@ -170,5 +167,5 @@
       <update_rate>20</update_rate>
       <topic>scan</topic>
-      <!- Header frame id used in gz msgs; bridge to ROS if needed ->
+      <!-- Header frame id used in gz msgs; bridge to ROS if needed -->
       <frame_id>base_scan</frame_id>
       <gz_frame_id>base_scan</gz_frame_id>
@@ -181,4 +178,10 @@
             <max_angle>3.14</max_angle>
           </horizontal>
+          <vertical>
+            <samples>8</samples>
+            <resolution>1</resolution>
+            <min_angle>-0.261799</min_angle>
+            <max_angle>0.0</max_angle>
+          </vertical>
         </scan>
         <range>
@@ -192,5 +195,5 @@
       </ros>
     </sensor>
-  </gazebo> -->
+  </gazebo>
 <gazebo reference="left_camera_frame">
     <sensor name="left_camera" type="camera">

File: ROS_ws/src/custom_slam/urdf/osr_full.urdf.xacro (robot description, xacro)
@@ -421,10 +421,10 @@
         </joint>
     <link name="imu_link"></link>
-    <!-- <joint name="lidar_joint" type="fixed">
+    <joint name="lidar_joint" type="fixed">
         <parent link="base_link"/>
         <child link="base_scan"/>
         <origin xyz="0 0 0" rpy="0 0 0"/>
-    </joint> -->
-    <!-- <link name="base_scan"></link> -->
+    </joint>
+    <link name="base_scan"></link>
     <joint name="camera_joint" type="fixed">
         <parent link="base_link"/>
