Commit message: full pipeline with working global reloc

File: ROS_ws/src/custom_slam/urdf/gazebo.urdf.xacro (robot description, xacro)
@@ -126,4 +126,20 @@
         <state_interface name="velocity"/>
         <state_interface name="effort"/>
+    </joint>
+    <joint name="arm_rotate_join_L">
+        <state_interface name="position"/>
+        <state_interface name="velocity"/>
+    </joint>
+    <joint name="arm_rotate_join_R">
+        <state_interface name="position"/>
+        <state_interface name="velocity"/>
+    </joint>
+    <joint name="body_axis_joint_L">
+        <state_interface name="position"/>
+        <state_interface name="velocity"/>
+    </joint>
+    <joint name="body_axis_joint_R">
+        <state_interface name="position"/>
+        <state_interface name="velocity"/>
     </joint>
   </ros2_control>
@@ -156,16 +172,14 @@
       <gz_frame_id>imu_link</gz_frame_id>
       <frame_id>imu_link</frame_id>
-      <!-- Optional: orientation reference / noise can be added here -->
     </sensor>
   </gazebo>
   <!-- GPU LiDAR on lidar_link -->
-  <gazebo reference="base_scan">
+  <!-- <gazebo reference="base_scan">
     <sensor type="gpu_lidar" name="lidar_sensor">
       <always_on>true</always_on>
       <visualize>true</visualize>
       <pose>-0.064 0 0.121 0 0 0</pose>
-      <update_rate>20</update_rate>
+      <update_rate>5</update_rate>
       <topic>scan</topic>
-      <!-- Header frame id used in gz msgs; bridge to ROS if needed -->
       <frame_id>base_scan</frame_id>
       <gz_frame_id>base_scan</gz_frame_id>
@@ -173,5 +187,5 @@
         <scan>
           <horizontal>
-            <samples>360</samples>
+            <samples>180</samples>
             <resolution>1</resolution>
             <min_angle>-3.14</min_angle>
@@ -195,9 +209,9 @@
       </ros>
     </sensor>
-  </gazebo>
+  </gazebo> -->
 <gazebo reference="left_camera_frame">
     <sensor name="left_camera" type="camera">
         <always_on>true</always_on>
-        <update_rate>30</update_rate>
+        <update_rate>20</update_rate>
         <topic>left_camera/image_raw</topic>
         <gz_frame_id>left_camera_optical_frame</gz_frame_id>
@@ -220,5 +234,5 @@
     <sensor name="right_camera" type="camera">
         <always_on>true</always_on>
-        <update_rate>30</update_rate>
+        <update_rate>20</update_rate>
         <topic>right_camera/image_raw</topic>
         <gz_frame_id>right_camera_optical_frame</gz_frame_id>

File: ROS_ws/src/custom_slam/urdf/osr_full.urdf.xacro (robot description, xacro)
@@ -93,9 +93,11 @@
             </inertial>
         </link>
-        <joint name="arm_rotate_join_${prefix}" type="fixed">
+        <joint name="arm_rotate_join_${prefix}" type="revolute">
             <parent link="box_rotate"/>
             <origin rpy="0 0.0 0" xyz="0 ${dir*0.153} 0"/>
             <child link="arm_rotate_${prefix}"/>
             <axis xyz="0 1 0"/>
+            <limit effort="0" velocity="1.0" lower="-0.3" upper="0.3"/>
+            <dynamics damping="0.5" friction="0.1"/>
         </joint>
     </xacro:macro>
@@ -127,5 +129,7 @@
             <origin rpy="0 0 0" xyz="0.071558 ${dir*0.017545} -0.084292"/>
             <child link="turn_bukles_link_${prefix}"/>
-            <axis xyz="0 1 0"/>
+            <!-- <axis xyz="0 1 0"/>
+            <limit effort="0" velocity="1.0" lower="-0.3" upper="0.3"/>
+            <dynamics damping="0.5" friction="0.1"/> -->
         </joint>
     </xacro:macro>
@@ -153,9 +157,11 @@
             </inertial>
         </link>
-        <joint name="body_axis_joint_${prefix}" type="fixed">
+        <joint name="body_axis_joint_${prefix}" type="revolute">
             <parent link="turn_bukles_link_${prefix}"/>
             <origin rpy="0 0 0" xyz="0 ${dir*-0.060920} -0.001245"/>
             <child link="body_axis_link_${prefix}"/>
             <axis xyz="0 1 0"/>
+            <limit effort="0" velocity="1.0" lower="-0.3" upper="0.3"/>
+            <dynamics damping="0.5" friction="0.1"/>
         </joint>
     </xacro:macro>
@@ -187,6 +193,7 @@
             <origin rpy="0 0 0" xyz="0.016004 ${dir*0.071485} 0.001353"/>
             <child link="rocker_bogie_link_${prefix}_1"/>
-            <limit effort="10000.0" velocity="0.5" lower="-0.5" upper="0.5"/>
-            <axis xyz="0 1 0"/>
+            <!-- <limit effort="0" velocity="1.0" lower="-0.5" upper="0.5"/>
+            <axis xyz="0 1 0"/>
+            <dynamics damping="0.5" friction="0.1"/> -->
         </joint>
         <link name="rocker_bogie_link_${prefix}_2">
@@ -489,70 +496,3 @@
     </joint>
     <link name="right_camera_optical_frame"/>
-    <!-- <ros2_control name="RobotSystem" type="system">
-        <hardware>
-            <plugin>gz_ros2_control/GazeboSimSystem</plugin>
-        </hardware>
-        <joint name="rear_wheel_joint_right">
-            <command_interface name="velocity"/>
-            <state_interface name="position"/>
-            <state_interface name="velocity"/>
-        </joint>
-        <joint name="rear_wheel_joint_left">
-            <command_interface name="velocity"/>
-            <state_interface name="position"/>
-            <state_interface name="velocity"/>
-        </joint>
-        <joint name="middle_wheel_joint_right">
-            <command_interface name="velocity"/>
-            <state_interface name="position"/>
-            <state_interface name="velocity"/>
-        </joint>
-        <joint name="middle_wheel_joint_left">
-            <command_interface name="velocity"/>
-            <state_interface name="position"/>
-            <state_interface name="velocity"/>
-        </joint>
-        <joint name="front_wheel_joint_right">
-            <command_interface name="velocity"/>
-            <state_interface name="position"/>
-            <state_interface name="velocity"/>
-        </joint>
-        <joint name="front_wheel_joint_left">
-            <command_interface name="velocity"/>
-            <state_interface name="position"/>
-            <state_interface name="velocity"/>
-        </joint>
-        <joint name="front_wheel_joint_R">
-            <command_interface name="position"/>
-            <state_interface name="position"/>
-            <state_interface name="velocity"/>
-        </joint>
-        <joint name="front_wheel_joint_L">
-            <command_interface name="position"/>
-            <state_interface name="position"/>
-            <state_interface name="velocity"/>
-        </joint>
-        <joint name="rear_wheel_joint_R">
-            <command_interface name="position"/>
-            <state_interface name="position"/>
-            <state_interface name="velocity"/>
-        </joint>
-        <joint name="rear_wheel_joint_L">
-            <command_interface name="position"/>
-            <state_interface name="position"/>
-            <state_interface name="velocity"/>
-        </joint>
-        <joint name="rocker_bogie_joint_L_2">
-            <command_interface name="effort"/>
-            <state_interface name="position"/>
-            <state_interface name="velocity"/>
-            <state_interface name="effort"/>
-        </joint>
-        <joint name="rocker_bogie_joint_R_2">
-            <command_interface name="effort"/>
-            <state_interface name="position"/>
-            <state_interface name="velocity"/>
-            <state_interface name="effort"/>
-        </joint>
-    </ros2_control> -->
 </robot>
